Commit message: updated hardware limits

File: models/icub_heidelberg01_no_weights.urdf (robot description, URDF)
Before this commit: robot iCubHeidelberg01_SIM_MODEL, 23 links, 22 joints
Joints:
- joint l_ankle_pitch: limit lower=-0.349065850399 upper=0.523598775598 effort=50000 velocity=50000 -> lower=-0.349065850399 upper=0.471238898 effort=50000 velocity=50000
- joint l_hip_pitch: limit lower=-0.523598775598 upper=1.4835298642 effort=50000 velocity=50000 -> lower=-0.34906585 upper=1.047197551 effort=50000 velocity=50000
- joint l_hip_roll: limit lower=0.0 upper=1.57079632679 effort=50000 velocity=50000 -> lower=0.0 upper=0.453785606 effort=50000 velocity=50000
- joint l_hip_yaw: limit lower=-1.2217304764 upper=1.2217304764 effort=50000 velocity=50000 -> lower=-0.872664626 upper=0.872664626 effort=50000 velocity=50000
- joint r_ankle_pitch: limit lower=-0.349065850399 upper=0.523598775598 effort=50000 velocity=50000 -> lower=-0.349065850399 upper=0.471238898 effort=50000 velocity=50000
- joint r_hip_pitch: limit lower=-0.523598775598 upper=1.4835298642 effort=50000 velocity=50000 -> lower=-0.34906585 upper=1.047197551 effort=50000 velocity=50000
- joint r_hip_roll: limit lower=0.0 upper=1.57079632679 effort=50000 velocity=50000 -> lower=0.0 upper=0.453785606 effort=50000 velocity=50000
- joint r_hip_yaw: limit lower=-1.2217304764 upper=1.2217304764 effort=50000 velocity=50000 -> lower=-0.872664626 upper=0.872664626 effort=50000 velocity=50000
- joint torso_pitch: limit lower=-0.349065850399 upper=1.2217304764 effort=50000 velocity=50000 -> lower=-0.349065850399 upper=1.047197551 effort=50000 velocity=50000
- joint torso_roll: limit lower=-0.523598775598 upper=0.523598775598 effort=50000 velocity=50000 -> lower=-0.453785606 upper=0.453785606 effort=50000 velocity=50000

Commit message: removed asymmetry

File: models/icub_heidelberg01_no_weights.urdf (robot description, URDF)
Before this commit: robot iCubHeidelberg01_SIM_MODEL, 23 links, 22 joints
Joints:
- joint l_ankle_pitch: axis -1.0 -0.0 -0.0 -> -1.0 0.0 0.0; origin xyz=-0.021343 -0.200983719847 0.00294927094483 rpy=2.4080004131e-05 0 0 -> xyz=-0.021343 -0.201 0.0 rpy=2.40788999988e-05 0 0
- joint l_ankle_roll: axis -0.0 0 -1 -> 0.0 0.0 -1.0; origin xyz=0.0355 -1.6398477099e-05 -0.0475117797388 rpy=0 0 0 -> xyz=0.0355 0.0 -0.0445624670112 rpy=0 0 0
- joint l_hip_roll: axis -0.0 0 -1 -> 0.0 0.0 -1.0; origin xyz=-0.059 -8.59963575406e-07 0.026362200929 rpy=0 0 0 -> xyz=-0.059 0 0.0263622 rpy=0 0 0
- joint l_hip_yaw: axis -0.0 1 0 -> 0.0 1.0 0.0; origin xyz=0.000121 0 0.017999 rpy=-1.5640768048 0 1.57079632679 -> xyz=0.0 0 0.018 rpy=-1.57079632679 0 1.57079632679
- joint l_knee: origin xyz=-0.017957 -0.145625287455 0 rpy=0 0 0 -> xyz=-0.017957 -0.145625 0 rpy=0 0 0
- joint l_leg_ft_sensor: origin xyz=0 -0.0743000549473 -0.0255046186937 rpy=0 1.5640768048 -1.57079632679 -> xyz=0 -0.0743 -0.0255047 rpy=0 1.5640768048 -1.57079632679
- joint r_ankle_pitch: origin xyz=-0.021343 -0.201 0 rpy=-2.40788999988e-05 0 0 -> xyz=-0.021343 -0.201 0.0 rpy=-2.40788999988e-05 0 0
- joint r_ankle_roll: axis -0.0 0 -1.0 -> 0.0 0.0 -1.0; origin xyz=0.0355 0 0.0445624670112 rpy=0 0 0 -> xyz=0.0355 0.0 0.0445624670112 rpy=0 0 0
